File: power.kicad_sch (KiCad schematic)
At the start: 0 parts

Commit message: Design power
Parts:
- added Boost: TPS610333DRLR, DRL0008A-MFG, symbol TPS610333DRLR:TPS610333DRLR
- added Current_Monitor: MCP3204T-CI/SL, SOIC14-N_MC_MCH, symbol MCP3204T_CI_SL:MCP3204T-CI_SL
- added L_{Boost}: 1uH, symbol Device:L
- added SYS_BYPASS, VIN_BYPASS: 1mF, symbol Device:C_Polarized
- added USB_Default_Power_CC1, USB_Default_Power_CC2: 5.1K, symbol Device:R_US
- added VBUS_SEL: 1N4148WX-TP, Diode_SMD:D_SOD-323, symbol Diode:1N4148W
- added Wired_Interface: USB4105-GF-A, USB4105-GF-A:GCT_USB4105-GF-A, symbol USB4105-GF-A:USB4105-GF-A
Connections:
- new net: Current_Monitor.2 (CH1), USB_Default_Power_CC1.1, Wired_Interface.A5 (CC1)
- new net: Boost.7 (SW), L_{Boost}.2
- new net: Current_Monitor.1 (CH0), USB_Default_Power_CC2.1, Wired_Interface.B5 (CC2)
- new net Battery/CHRG_DIV: Current_Monitor.4 (CH3)
- new net Battery/V_{BAT}: Boost.1 (VIN), Boost.2 (EN), Boost.5 (FB), L_{Boost}.1, VBUS_SEL.1 (K), VIN_BYPASS.1
- new net Battery/V_{BUS}: VBUS_SEL.2 (A), Wired_Interface.A4_B9 (VBUS), Wired_Interface.B4_A9 (VBUS)
- new net Battery/V_{LDO}: Current_Monitor.13 (VREF), Current_Monitor.14 (VDD)
- new net CLK_{Current}: Current_Monitor.11 (CLK)
- new net CS_{Current}: Current_Monitor.8 (*CS/SHDN)
- new net DIN_{Current}: Current_Monitor.9 (DIN)
- new net DOUT_{Current}: Current_Monitor.10 (DOUT)
- new net Data_Negative: Wired_Interface.A7 (DN1), Wired_Interface.B7 (DN2)
- new net Data_Positive: Wired_Interface.A6 (DP1), Wired_Interface.B6 (DP2)
- new net GND: Boost.3 (MODE), Boost.6 (GND), Current_Monitor.12 (AGND), Current_Monitor.7 (DGND), SYS_BYPASS.2, USB_Default_Power_CC1.2, USB_Default_Power_CC2.2, VIN_BYPASS.2, Wired_Interface.A1_B12 (GND), Wired_Interface.B1_A12 (GND), Wired_Interface.SH1 (SHELL_GND), Wired_Interface.SH2 (SHELL_GND), Wired_Interface.SH3 (SHELL_GND), Wired_Interface.SH4 (SHELL_GND)
- new net V_{SYS}: Boost.8 (VOUT), SYS_BYPASS.1
- no-connect marks 0 -> 6
Other:
- added sheet Battery (battery.kicad_sch)
- title: Port Plover -> Stenoswitch
