File: battery.kicad_sch (KiCad schematic)
At the start: 38 parts

Commit message: Rework right hand
Parts:
- renumbered C_{BATT}1 to C_{BATT}0, C_{BATT}0 to C_{BATT}1
Changed lines of the file:
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@@
 		(dnp no)
 		(fields_autoplaced yes)
-		(property "Reference" "#PWR012"
+		(property "Reference" "#PWR030"
 			(at 181.61 147.32 0)
 			(effects
@@
 		(dnp no)
 		(fields_autoplaced yes)
-		(property "Reference" "#PWR04"
+		(property "Reference" "#PWR021"
 			(at 85.09 121.92 0)
 			(effects
@@
 		(dnp no)
 		(fields_autoplaced yes)
-		(property "Reference" "#PWR011"
+		(property "Reference" "#PWR013"
 			(at 157.48 111.76 0)
 			(effects
@@
 		(dnp no)
 		(fields_autoplaced yes)
-		(property "Reference" "#PWR018"
+		(property "Reference" "#PWR024"
 			(at 232.41 97.79 0)
 			(effects
@@
 		(dnp no)
 		(fields_autoplaced yes)
-		(property "Reference" "#PWR00"
+		(property "Reference" "#PWR027"
 			(at 40.64 92.71 0)
 			(effects
@@
 		(dnp no)
 		(fields_autoplaced yes)
-		(property "Reference" "#PWR08"
+		(property "Reference" "#PWR018"
 			(at 135.89 63.5 0)
 			(effects
@@
 		(dnp no)
 		(fields_autoplaced yes)
-		(property "Reference" "#PWR016"
+		(property "Reference" "#PWR012"
 			(at 214.63 100.33 0)
 			(effects
@@
 		(dnp no)
 		(fields_autoplaced yes)
-		(property "Reference" "#PWR017"
+		(property "Reference" "#PWR023"
 			(at 217.17 132.08 0)
 			(effects
@@
 		(on_board yes)
 		(dnp no)
-		(property "Reference" "#PWR07"
+		(property "Reference" "#PWR025"
 			(at 115.57 125.73 0)
 			(effects
@@
 		(dnp no)
 		(fields_autoplaced yes)
-		(property "Reference" "#PWR013"
+		(property "Reference" "#PWR010"
 			(at 190.5 102.87 0)
 			(effects
@@
 		(dnp no)
 		(fields_autoplaced yes)
-		(property "Reference" "#PWR014"
+		(property "Reference" "#PWR031"
 			(at 194.31 147.32 0)
 			(effects
@@
 		(dnp no)
 		(fields_autoplaced yes)
-		(property "Reference" "#PWR01"
+		(property "Reference" "#PWR016"
 			(at 55.88 68.58 0)
 			(effects
@@
 		(on_board yes)
 		(dnp no)
-		(property "Reference" "C_{BATT}1"
+		(property "Reference" "C_{BATT}0"
 			(at 52.07 81.2799 0)
 			(effects
@@
 		(dnp no)
 		(fields_autoplaced yes)
-		(property "Reference" "#PWR010"
+		(property "Reference" "#PWR019"
 			(at 156.21 181.61 0)
 			(effects
@@
 		(dnp no)
 		(fields_autoplaced yes)
-		(property "Reference" "#PWR015"
+		(property "Reference" "#PWR028"
 			(at 208.28 147.32 0)
 			(effects
@@
 		(on_board yes)
 		(dnp no)
-		(property "Reference" "C_{BATT}0"
+		(property "Reference" "C_{BATT}1"
 			(at 36.83 81.2799 0)
 			(effects
@@
 		(dnp no)
 		(fields_autoplaced yes)
-		(property "Reference" "#PWR019"
+		(property "Reference" "#PWR029"
 			(at 250.19 90.17 0)
 			(effects
@@
 		(dnp no)
 		(fields_autoplaced yes)
-		(property "Reference" "#PWR02"
+		(property "Reference" "#PWR022"
 			(at 55.88 92.71 0)
 			(effects
@@
 		(dnp no)
 		(fields_autoplaced yes)
-		(property "Reference" "#PWR03"
+		(property "Reference" "#PWR026"
 			(at 66.04 107.95 0)
 			(effects
@@
 		(dnp no)
 		(fields_autoplaced yes)
-		(property "Reference" "#PWR05"
+		(property "Reference" "#PWR09"
 			(at 91.44 116.84 0)
 			(effects
@@
 		(dnp no)
 		(fields_autoplaced yes)
-		(property "Reference" "#PWR09"
+		(property "Reference" "#PWR020"
 			(at 142.24 60.96 0)
 			(effects
@@
 		(dnp no)
 		(fields_autoplaced yes)
-		(property "Reference" "#PWR06"
+		(property "Reference" "#PWR017"
 			(at 111.76 195.58 0)
 			(effects

Commit message: Update layout
Parts:
- BAT0: footprint BAT_1043 -> 1043:BAT_1043; symbol 1042:1042 -> 1043:1043; MAXIMUM_PACKAGE_HEIGHT 15.11mm -> 14.86mm; PARTREV E -> J; SNAPEDA_PN 1042 -> 1043
- Battery_Monitor0: footprint IC_BQ27427YZFR -> BQ27427YZFR:IC_BQ27427YZFR
Connections:
- net at Battery_Monitor0.B1 (BIN): now also BAT_EN0.1, Battery_Charger0.5 (BATT), CHRG_Shunt0.1, C_{BATT}0.1, C_{BATT}1.1; no longer BIN_Pulldown0.2
- new net: BIN_Pulldown0.2, Battery_Monitor0.C2 (SRX)
Changed lines of the file:
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@@
 	)
 	(junction
-		(at 114.3 119.38)
-		(diameter 0)
-		(color 0 0 0 0)
-	)
-	(junction
 		(at 111.76 182.88)
 		(diameter 0)
@@
 	)
 	(junction
-		(at 165.1 149.86)
+		(at 115.57 119.38)
 		(diameter 0)
 		(color 0 0 0 0)
 	)
 	(junction
-		(at 208.28 133.35)
+		(at 165.1 149.86)
 		(diameter 0)
 		(color 0 0 0 0)
 	)
 	(junction
-		(at 115.57 119.38)
+		(at 208.28 133.35)
 		(diameter 0)
 		(color 0 0 0 0)
@@
 	)
 	(junction
-		(at 144.78 149.86)
+		(at 116.84 119.38)
 		(diameter 0)
 		(color 0 0 0 0)
 	)
 	(junction
-		(at 116.84 119.38)
+		(at 144.78 149.86)
 		(diameter 0)
 		(color 0 0 0 0)
@@
 	)
 	(junction
+		(at 114.3 119.38)
+		(diameter 0)
+		(color 0 0 0 0)
+	)
+	(junction
 		(at 250.19 76.2)
 		(diameter 0)
@@
 	(wire
 		(pts
-			(xy 85.09 107.95) (xy 91.44 107.95)
-		)
-		(stroke
-			(width 0)
-			(type default)
-		)
-	)
-	(wire
-		(pts
-			(xy 111.76 119.38) (xy 114.3 119.38)
-		)
-		(stroke
-			(width 0)
-			(type default)
-		)
-	)
-	(wire
-		(pts
 			(xy 91.44 154.94) (xy 91.44 149.86)
 		)
@@
 	(wire
 		(pts
+			(xy 85.09 107.95) (xy 91.44 107.95)
+		)
+		(stroke
+			(width 0)
+			(type default)
+		)
+	)
+	(wire
+		(pts
 			(xy 165.1 149.86) (xy 165.1 160.02)
 		)
@@
 	(wire
 		(pts
-			(xy 114.3 119.38) (xy 115.57 119.38)
+			(xy 68.58 44.45) (xy 83.82 44.45)
 		)
 		(stroke
@@
 	(wire
 		(pts
-			(xy 68.58 44.45) (xy 83.82 44.45)
+			(xy 63.5 76.2) (xy 67.31 76.2)
 		)
 		(stroke
@@
 	(wire
 		(pts
-			(xy 63.5 76.2) (xy 67.31 76.2)
+			(xy 168.91 149.86) (xy 165.1 149.86)
 		)
 		(stroke
@@
 	(wire
 		(pts
-			(xy 168.91 149.86) (xy 165.1 149.86)
+			(xy 115.57 119.38) (xy 116.84 119.38)
 		)
 		(stroke
@@
 	(wire
 		(pts
-			(xy 116.84 119.38) (xy 119.38 119.38)
-		)
-		(stroke
-			(width 0)
-			(type default)
-		)
-	)
-	(wire
-		(pts
 			(xy 55.88 36.83) (xy 83.82 36.83)
 		)
@@
 	(wire
 		(pts
+			(xy 114.3 119.38) (xy 115.57 119.38)
+		)
+		(stroke
+			(width 0)
+			(type default)
+		)
+	)
+	(wire
+		(pts
 			(xy 63.5 41.91) (xy 83.82 41.91)
 		)
@@
 	(wire
 		(pts
-			(xy 115.57 119.38) (xy 116.84 119.38)
+			(xy 111.76 119.38) (xy 114.3 119.38)
 		)
 		(stroke
@@
 	(wire
 		(pts
+			(xy 116.84 119.38) (xy 119.38 119.38)
+		)
+		(stroke
+			(width 0)
+			(type default)
+		)
+	)
+	(wire
+		(pts
 			(xy 68.58 64.77) (xy 68.58 44.45)
 		)
@@
 			)
 		)
-		(property "Footprint" "IC_BQ27427YZFR"
+		(property "Footprint" "BQ27427YZFR:IC_BQ27427YZFR"
 			(at 99.06 44.45 0)
 			(effects
@@
 	)
 	(symbol
+		(lib_name "C_1")
 		(lib_id "Device:C")
 		(at 190.5 92.71 0)
@@
 				)
 			)
-			(project "right_hand"
-				(path "/efcccfe8-5e20-4b1b-8d3b-61fce771481e/cd3314d0-f605-42f0-be2b-644cabc7637c/acaa3521-7032-4a8a-adbb-019f51b56731"
-					(reference "CHRG_Decouple0")
-					(unit 1)
-				)
-			)
 		)
 	)
@@
 		(dnp no)
 		(fields_autoplaced yes)
-		(property "Reference" "#PWR016"
+		(property "Reference" "#PWR01"
 			(at 55.88 68.58 0)
 			(effects
@@
 			(project "portable_steno"
 				(path "/06a6eca0-edda-4cc0-a23f-017602e67f07/99f3b279-b2b0-4dd5-ab05-9b518546ce95/cd3314d0-f605-42f0-be2b-644cabc7637c/acaa3521-7032-4a8a-adbb-019f51b56731"
-					(reference "#PWR016")
-					(unit 1)
-				)
-			)
-			(project "right_hand"
-				(path "/efcccfe8-5e20-4b1b-8d3b-61fce771481e/cd3314d0-f605-42f0-be2b-644cabc7637c/acaa3521-7032-4a8a-adbb-019f51b56731"
 					(reference "#PWR01")
 					(unit 1)
@@
 	)
 	(symbol
+		(lib_name "R_US_1")
 		(lib_id "Device:R_US")
 		(at 85.09 111.76 0)
@@
 				)
 			)
-			(project "right_hand"
-				(path "/efcccfe8-5e20-4b1b-8d3b-61fce771481e/cd3314d0-f605-42f0-be2b-644cabc7637c/acaa3521-7032-4a8a-adbb-019f51b56731"
-					(reference "R_{ISET}0")
-					(unit 1)
-				)
-			)
 		)
 	)
@@
 	)
 	(symbol
+		(lib_name "R_US_2")
 		(lib_id "Device:R_US")
 		(at 171.45 101.6 0)
@@
 	)
 	(symbol
+		(lib_name "R_US_3")
 		(lib_id "Device:R_US")
 		(at 149.86 105.41 270)
@@
 	)
 	(symbol
+		(lib_name "R_Small_US_1")
 		(lib_id "Device:R_Small_US")
 		(at 157.48 102.87 0)
@@
 				)
 			)
-			(project "right_hand"
-				(path "/efcccfe8-5e20-4b1b-8d3b-61fce771481e/cd3314d0-f605-42f0-be2b-644cabc7637c/acaa3521-7032-4a8a-adbb-019f51b56731"
-					(reference "BAT_Fuse0")
-					(unit 1)
-				)
-			)
 		)
 	)
@@
 	)
 	(symbol
-		(lib_id "1042:1042")
+		(lib_id "1043:1043")
 		(at 55.88 54.61 270)
 		(unit 1)
@@
 			)
 		)
-		(property "Footprint" "BAT_1043"
+		(property "Footprint" "1043:BAT_1043"
 			(at 55.88 54.61 0)
 			(effects
@@
 			)
 		)
-		(property "PARTREV" "E"
+		(property "PARTREV" "J"
 			(at 55.88 54.61 0)
 			(effects
@@
 			)
 		)
-		(property "SNAPEDA_PN" "1042"
+		(property "SNAPEDA_PN" "1043"
 			(at 55.88 54.61 0)
 			(effects
@@
 			)
 		)
-		(property "MAXIMUM_PACKAGE_HEIGHT" "15.11mm"
+		(property "MAXIMUM_PACKAGE_HEIGHT" "14.86mm"
 			(at 55.88 54.61 0)
 			(effects
