File: control.kicad_sch (KiCad schematic)
At the start: 4 parts

Commit message: Replace USB connector
Parts:
- renumbered BT_EN0 to BT_EN1, STORAGE_EN0 to STORAGE_EN1, TRANSLATION_EN0 to TRANSLATION_EN1
Changed lines of the file:
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@@
 		(dnp no)
 		(fields_autoplaced yes)
-		(property "Reference" "#PWR034"
+		(property "Reference" "#PWR020"
 			(at 144.78 80.01 0)
 			(effects
@@
 		(dnp no)
 		(fields_autoplaced yes)
-		(property "Reference" "TRANSLATION_EN0"
+		(property "Reference" "TRANSLATION_EN1"
 			(at 176.53 38.1 0)
 			(effects
@@
 		(dnp no)
 		(fields_autoplaced yes)
-		(property "Reference" "#PWR06"
+		(property "Reference" "#PWR025"
 			(at 63.5 49.53 0)
 			(effects
@@
 		(dnp no)
 		(fields_autoplaced yes)
-		(property "Reference" "STORAGE_EN0"
+		(property "Reference" "STORAGE_EN1"
 			(at 175.26 59.69 0)
 			(effects
@@
 		(dnp no)
 		(fields_autoplaced yes)
-		(property "Reference" "#PWR014"
+		(property "Reference" "#PWR0127"
 			(at 182.88 76.2 0)
 			(effects
@@
 		(dnp no)
 		(fields_autoplaced yes)
-		(property "Reference" "#PWR032"
+		(property "Reference" "#PWR024"
 			(at 73.66 54.61 0)
 			(effects
@@
 		(dnp no)
 		(fields_autoplaced yes)
-		(property "Reference" "BT_EN0"
+		(property "Reference" "BT_EN1"
 			(at 175.26 80.01 0)
 			(effects
@@
 		(dnp no)
 		(fields_autoplaced yes)
-		(property "Reference" "#PWR033"
+		(property "Reference" "#PWR026"
 			(at 142.24 59.69 0)
 			(effects
@@
 		(dnp no)
 		(fields_autoplaced yes)
-		(property "Reference" "#PWR00"
+		(property "Reference" "#PWR0128"
 			(at 182.88 96.52 0)
 			(effects
@@
 		(dnp no)
 		(fields_autoplaced yes)
-		(property "Reference" "#PWR011"
+		(property "Reference" "#PWR022"
 			(at 69.85 74.93 0)
 			(effects
@@
 		(dnp no)
 		(fields_autoplaced yes)
-		(property "Reference" "#PWR015"
+		(property "Reference" "#PWR0126"
 			(at 184.15 54.61 0)
 			(effects
