File: left_hand_keys.kicad_sch (KiCad schematic)
At the start: 40 parts

Commit message: Label keys
Parts:
- renumbered Key25 to A, Key26 to Asterisk0, Key27 to Asterisk1, Key23 to H, Key20 to K, Number_Bar6 to Number_Bar0, Number_Bar7 to Number_Bar1, Number_Bar8 to Number_Bar2, Number_Bar9 to Number_Bar3, Number_Bar10 to Number_Bar4, Number_Bar11 to Number_Bar5, Key28 to O, Key21 to P, Key24 to R, Key17 to S0, Key18 to S1, Key15 to Spare0, Key16 to Spare1, Key19 to T, Key22 to W
Changed lines of the file:
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@@
 		(dnp no)
 		(fields_autoplaced yes)
-		(property "Reference" "Number_Bar9"
+		(property "Reference" "Number_Bar3"
 			(at 152.4 50.8 0)
 			(effects
@@
 			(project "portable_steno"
 				(path "/06a6eca0-edda-4cc0-a23f-017602e67f07/2477db2d-d681-4372-a745-e817369fb274/f651b724-284b-4a82-a638-8f4a85d8d53c"
-					(reference "Number_Bar9")
+					(reference "Number_Bar3")
 					(unit 1)
 				)
@@
 		(on_board yes)
 		(dnp no)
-		(property "Reference" "Key15"
+		(property "Reference" "Spare0"
 			(at 30.48 72.39 0)
 			(effects
@@
 			(project "portable_steno"
 				(path "/06a6eca0-edda-4cc0-a23f-017602e67f07/2477db2d-d681-4372-a745-e817369fb274/f651b724-284b-4a82-a638-8f4a85d8d53c"
-					(reference "Key15")
+					(reference "Spare0")
 					(unit 1)
 				)
@@
 		(on_board yes)
 		(dnp no)
-		(property "Reference" "Key21"
+		(property "Reference" "P"
 			(at 152.4 72.39 0)
 			(effects
@@
 			(project "portable_steno"
 				(path "/06a6eca0-edda-4cc0-a23f-017602e67f07/2477db2d-d681-4372-a745-e817369fb274/f651b724-284b-4a82-a638-8f4a85d8d53c"
-					(reference "Key21")
+					(reference "P")
 					(unit 1)
 				)
@@
 		(on_board yes)
 		(dnp no)
-		(property "Reference" "Key20"
+		(property "Reference" "K"
 			(at 111.76 93.98 0)
 			(effects
@@
 			(project "portable_steno"
 				(path "/06a6eca0-edda-4cc0-a23f-017602e67f07/2477db2d-d681-4372-a745-e817369fb274/f651b724-284b-4a82-a638-8f4a85d8d53c"
-					(reference "Key20")
+					(reference "K")
 					(unit 1)
 				)
@@
 		(dnp no)
 		(fields_autoplaced yes)
-		(property "Reference" "Number_Bar8"
+		(property "Reference" "Number_Bar2"
 			(at 110.49 50.8 0)
 			(effects
@@
 			(project "portable_steno"
 				(path "/06a6eca0-edda-4cc0-a23f-017602e67f07/2477db2d-d681-4372-a745-e817369fb274/f651b724-284b-4a82-a638-8f4a85d8d53c"
-					(reference "Number_Bar8")
+					(reference "Number_Bar2")
 					(unit 1)
 				)
@@
 		(on_board yes)
 		(dnp no)
-		(property "Reference" "Key16"
+		(property "Reference" "Spare1"
 			(at 30.48 93.98 0)
 			(effects
@@
 			(project "portable_steno"
 				(path "/06a6eca0-edda-4cc0-a23f-017602e67f07/2477db2d-d681-4372-a745-e817369fb274/f651b724-284b-4a82-a638-8f4a85d8d53c"
-					(reference "Key16")
+					(reference "Spare1")
 					(unit 1)
 				)
@@
 		(on_board yes)
 		(dnp no)
-		(property "Reference" "Key18"
+		(property "Reference" "S1"
 			(at 71.12 93.98 0)
 			(effects
@@
 			(project "portable_steno"
 				(path "/06a6eca0-edda-4cc0-a23f-017602e67f07/2477db2d-d681-4372-a745-e817369fb274/f651b724-284b-4a82-a638-8f4a85d8d53c"
-					(reference "Key18")
+					(reference "S1")
 					(unit 1)
 				)
@@
 		(on_board yes)
 		(dnp no)
-		(property "Reference" "Key25"
+		(property "Reference" "A"
 			(at 193.04 115.57 0)
 			(effects
@@
 			(project "portable_steno"
 				(path "/06a6eca0-edda-4cc0-a23f-017602e67f07/2477db2d-d681-4372-a745-e817369fb274/f651b724-284b-4a82-a638-8f4a85d8d53c"
-					(reference "Key25")
+					(reference "A")
 					(unit 1)
 				)
@@
 		(on_board yes)
 		(dnp no)
-		(property "Reference" "Key24"
+		(property "Reference" "R"
 			(at 193.04 93.98 0)
 			(effects
@@
 			(project "portable_steno"
 				(path "/06a6eca0-edda-4cc0-a23f-017602e67f07/2477db2d-d681-4372-a745-e817369fb274/f651b724-284b-4a82-a638-8f4a85d8d53c"
-					(reference "Key24")
+					(reference "R")
 					(unit 1)
 				)
@@
 		(on_board yes)
 		(dnp no)
-		(property "Reference" "Key22"
+		(property "Reference" "W"
 			(at 152.4 93.98 0)
 			(effects
@@
 			(project "portable_steno"
 				(path "/06a6eca0-edda-4cc0-a23f-017602e67f07/2477db2d-d681-4372-a745-e817369fb274/f651b724-284b-4a82-a638-8f4a85d8d53c"
-					(reference "Key22")
+					(reference "W")
 					(unit 1)
 				)
@@
 		(on_board yes)
 		(dnp no)
-		(property "Reference" "Key26"
+		(property "Reference" "Asterisk0"
 			(at 232.41 72.39 0)
 			(effects
@@
 			(project "portable_steno"
 				(path "/06a6eca0-edda-4cc0-a23f-017602e67f07/2477db2d-d681-4372-a745-e817369fb274/f651b724-284b-4a82-a638-8f4a85d8d53c"
-					(reference "Key26")
+					(reference "Asterisk0")
 					(unit 1)
 				)
@@
 		(dnp no)
 		(fields_autoplaced yes)
-		(property "Reference" "Number_Bar7"
+		(property "Reference" "Number_Bar1"
 			(at 72.39 50.8 0)
 			(effects
@@
 			(project "portable_steno"
 				(path "/06a6eca0-edda-4cc0-a23f-017602e67f07/2477db2d-d681-4372-a745-e817369fb274/f651b724-284b-4a82-a638-8f4a85d8d53c"
-					(reference "Number_Bar7")
+					(reference "Number_Bar1")
 					(unit 1)
 				)
@@
 		(on_board yes)
 		(dnp no)
-		(property "Reference" "Key27"
+		(property "Reference" "Asterisk1"
 			(at 232.41 93.98 0)
 			(effects
@@
 			(project "portable_steno"
 				(path "/06a6eca0-edda-4cc0-a23f-017602e67f07/2477db2d-d681-4372-a745-e817369fb274/f651b724-284b-4a82-a638-8f4a85d8d53c"
-					(reference "Key27")
+					(reference "Asterisk1")
 					(unit 1)
 				)
@@
 		(on_board yes)
 		(dnp no)
-		(property "Reference" "Key19"
+		(property "Reference" "T"
 			(at 111.76 72.39 0)
 			(effects
@@
 			(project "portable_steno"
 				(path "/06a6eca0-edda-4cc0-a23f-017602e67f07/2477db2d-d681-4372-a745-e817369fb274/f651b724-284b-4a82-a638-8f4a85d8d53c"
-					(reference "Key19")
+					(reference "T")
 					(unit 1)
 				)
@@
 		(on_board yes)
 		(dnp no)
-		(property "Reference" "Key17"
+		(property "Reference" "S0"
 			(at 71.12 72.39 0)
 			(effects
@@
 			(project "portable_steno"
 				(path "/06a6eca0-edda-4cc0-a23f-017602e67f07/2477db2d-d681-4372-a745-e817369fb274/f651b724-284b-4a82-a638-8f4a85d8d53c"
-					(reference "Key17")
+					(reference "S0")
 					(unit 1)
 				)
@@
 		(on_board yes)
 		(dnp no)
-		(property "Reference" "Key23"
+		(property "Reference" "H"
 			(at 193.04 72.39 0)
 			(effects
@@
 			(project "portable_steno"
 				(path "/06a6eca0-edda-4cc0-a23f-017602e67f07/2477db2d-d681-4372-a745-e817369fb274/f651b724-284b-4a82-a638-8f4a85d8d53c"
-					(reference "Key23")
+					(reference "H")
 					(unit 1)
 				)
@@
 		(on_board yes)
 		(dnp no)
-		(property "Reference" "Key28"
+		(property "Reference" "O"
 			(at 232.41 115.57 0)
 			(effects
@@
 			(project "portable_steno"
 				(path "/06a6eca0-edda-4cc0-a23f-017602e67f07/2477db2d-d681-4372-a745-e817369fb274/f651b724-284b-4a82-a638-8f4a85d8d53c"
-					(reference "Key28")
+					(reference "O")
 					(unit 1)
 				)
@@
 		(dnp no)
 		(fields_autoplaced yes)
-		(property "Reference" "Number_Bar6"
+		(property "Reference" "Number_Bar0"
 			(at 30.48 50.8 0)
 			(effects
@@
 			(project "portable_steno"
 				(path "/06a6eca0-edda-4cc0-a23f-017602e67f07/2477db2d-d681-4372-a745-e817369fb274/f651b724-284b-4a82-a638-8f4a85d8d53c"
-					(reference "Number_Bar6")
+					(reference "Number_Bar0")
 					(unit 1)
 				)
@@
 		(dnp no)
 		(fields_autoplaced yes)
-		(property "Reference" "Number_Bar11"
+		(property "Reference" "Number_Bar5"
 			(at 232.41 50.8 0)
 			(effects
@@
 			(project "portable_steno"
 				(path "/06a6eca0-edda-4cc0-a23f-017602e67f07/2477db2d-d681-4372-a745-e817369fb274/f651b724-284b-4a82-a638-8f4a85d8d53c"
-					(reference "Number_Bar11")
+					(reference "Number_Bar5")
 					(unit 1)
 				)
@@
 		(dnp no)
 		(fields_autoplaced yes)
-		(property "Reference" "Number_Bar10"
+		(property "Reference" "Number_Bar4"
 			(at 191.77 50.8 0)
 			(effects
@@
 			(project "portable_steno"
 				(path "/06a6eca0-edda-4cc0-a23f-017602e67f07/2477db2d-d681-4372-a745-e817369fb274/f651b724-284b-4a82-a638-8f4a85d8d53c"
-					(reference "Number_Bar10")
+					(reference "Number_Bar4")
 					(unit 1)
 				)

Commit message: Design power
Parts:
- D16, D17, D18, D19, D20, D21, D22, D23, D24, D25, D26, D27, D28, D29, D30, D32, D34, D36, D38, D40: footprint Diode_SMD:D_SOD-123 -> Diode_SMD:D_SOD-323
Other:
- title: Port Plover -> Stenoswitch
Changed lines of the file:
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@@
 	(paper "A4")
 	(title_block
-		(title "Port Plover")
-		(date "2025-07-28")
+		(title "Stenoswitch")
 		(rev "0.1")
 		(company "https://github.com/Bennett-Petzold/port_plover")
@@
 			)
 		)
-		(property "Footprint" "Diode_SMD:D_SOD-123"
+		(property "Footprint" "Diode_SMD:D_SOD-323"
 			(at 166.37 97.155 0)
 			(effects
@@
 			)
 		)
-		(property "Footprint" "Diode_SMD:D_SOD-123"
+		(property "Footprint" "Diode_SMD:D_SOD-323"
 			(at 166.37 75.565 0)
 			(effects
@@
 			)
 		)
-		(property "Footprint" "Diode_SMD:D_SOD-123"
+		(property "Footprint" "Diode_SMD:D_SOD-323"
 			(at 86.36 53.975 0)
 			(effects
@@
 			)
 		)
-		(property "Footprint" "Diode_SMD:D_SOD-123"
+		(property "Footprint" "Diode_SMD:D_SOD-323"
 			(at 207.01 75.565 0)
 			(effects
@@
 			)
 		)
-		(property "Footprint" "Diode_SMD:D_SOD-123"
+		(property "Footprint" "Diode_SMD:D_SOD-323"
 			(at 246.38 97.155 0)
 			(effects
@@
 			)
 		)
-		(property "Footprint" "Diode_SMD:D_SOD-123"
+		(property "Footprint" "Diode_SMD:D_SOD-323"
 			(at 44.45 75.565 0)
 			(effects
@@
 			)
 		)
-		(property "Footprint" "Diode_SMD:D_SOD-123"
+		(property "Footprint" "Diode_SMD:D_SOD-323"
 			(at 85.09 75.565 0)
 			(effects
@@
 			)
 		)
-		(property "Footprint" "Diode_SMD:D_SOD-123"
+		(property "Footprint" "Diode_SMD:D_SOD-323"
 			(at 166.37 53.975 0)
 			(effects
@@
 			)
 		)
-		(property "Footprint" "Diode_SMD:D_SOD-123"
+		(property "Footprint" "Diode_SMD:D_SOD-323"
 			(at 246.38 75.565 0)
 			(effects
@@
 			)
 		)
-		(property "Footprint" "Diode_SMD:D_SOD-123"
+		(property "Footprint" "Diode_SMD:D_SOD-323"
 			(at 125.73 97.155 0)
 			(effects
@@
 			)
 		)
-		(property "Footprint" "Diode_SMD:D_SOD-123"
+		(property "Footprint" "Diode_SMD:D_SOD-323"
 			(at 85.09 97.155 0)
 			(effects
@@
 			)
 		)
-		(property "Footprint" "Diode_SMD:D_SOD-123"
+		(property "Footprint" "Diode_SMD:D_SOD-323"
 			(at 125.73 75.565 0)
 			(effects
@@
 			)
 		)
-		(property "Footprint" "Diode_SMD:D_SOD-123"
+		(property "Footprint" "Diode_SMD:D_SOD-323"
 			(at 44.45 53.975 0)
 			(effects
@@
 			)
 		)
-		(property "Footprint" "Diode_SMD:D_SOD-123"
+		(property "Footprint" "Diode_SMD:D_SOD-323"
 			(at 246.38 53.975 0)
 			(effects
@@
 			)
 		)
-		(property "Footprint" "Diode_SMD:D_SOD-123"
+		(property "Footprint" "Diode_SMD:D_SOD-323"
 			(at 207.01 118.745 0)
 			(effects
@@
 			)
 		)
-		(property "Footprint" "Diode_SMD:D_SOD-123"
+		(property "Footprint" "Diode_SMD:D_SOD-323"
 			(at 124.46 53.975 0)
 			(effects
@@
 			)
 		)
-		(property "Footprint" "Diode_SMD:D_SOD-123"
+		(property "Footprint" "Diode_SMD:D_SOD-323"
 			(at 246.38 118.745 0)
 			(effects
@@
 			)
 		)
-		(property "Footprint" "Diode_SMD:D_SOD-123"
+		(property "Footprint" "Diode_SMD:D_SOD-323"
 			(at 207.01 97.155 0)
 			(effects
@@
 			)
 		)
-		(property "Footprint" "Diode_SMD:D_SOD-123"
+		(property "Footprint" "Diode_SMD:D_SOD-323"
 			(at 44.45 97.155 0)
 			(effects
@@
 			)
 		)
-		(property "Footprint" "Diode_SMD:D_SOD-123"
+		(property "Footprint" "Diode_SMD:D_SOD-323"
 			(at 205.74 53.975 0)
 			(effects

Commit message: Remove unnecessary diodes
Parts:
- removed D16, D21, D22, D25, D28, D34: 1N4148WX-TP, Diode_SMD:D_SOD-323, symbol Diode:1N4148W
- added D_{L}8: 1N4148WX-TP, Diode_SMD:D_SOD-323, symbol Diode:1N4148W
- renumbered A to A0, D17 to D_{L}0, D18 to D_{L}1, D30 to D_{L}10, D32 to D_{L}11, D36 to D_{L}12, D38 to D_{L}13, D40 to D_{L}14, D19 to D_{L}2, D20 to D_{L}3, D23 to D_{L}4, D24 to D_{L}5, D26 to D_{L}6, D27 to D_{L}7, D29 to D_{L}9, H to H0, K to K0, O to O0, P to P_{L}0, R to R_{L}0, T to T_{L}0, W to W0
Connections:
- net Columns2: now also D_{L}8.1 (K)
- net at Number_Bar3.2: now also Number_Bar0.2, Number_Bar1.2, Number_Bar2.2, Number_Bar4.2, Number_Bar5.2, D_{L}8.2 (A)

Commit message: Init right and left PCBs
Parts:
- renumbered A0 to A1, Asterisk0 to Asterisk1, Asterisk1 to Asterisk2, D_{L}0 to D_{L}1, D_{L}9 to D_{L}10, D_{L}10 to D_{L}11, D_{L}11 to D_{L}12, D_{L}12 to D_{L}13, D_{L}13 to D_{L}14, D_{L}14 to D_{L}15, D_{L}1 to D_{L}2, D_{L}2 to D_{L}3, D_{L}3 to D_{L}4, D_{L}4 to D_{L}5, D_{L}5 to D_{L}6, D_{L}6 to D_{L}7, D_{L}7 to D_{L}8, D_{L}8 to D_{L}9, H0 to H1, K0 to K1, Number_Bar0 to Number_Bar1, Number_Bar1 to Number_Bar2, Number_Bar2 to Number_Bar3, Number_Bar3 to Number_Bar4, Number_Bar4 to Number_Bar5, Number_Bar5 to Number_Bar6, O0 to O1, P_{L}0 to P_{L}1, R_{L}0 to R_{L}1, S0 to S1, S1 to S2, Spare0 to Spare1, Spare1 to Spare2, T_{L}0 to T_{L}1, W0 to W1

Commit message: Rename keyswitch diodes
Parts:
- renumbered D_{L}1 to D_{Spare}0

Commit message: Layout left hand side
Parts:
- renumbered A1 to A0, Asterisk1 to Asterisk0, Asterisk2 to Asterisk1, D_{L}14 to D_{AS}1, D_{L}13 to D_{As}0, D_{L}12 to D_{A}0, D_{L}10 to D_{H}0, D_{L}6 to D_{K}0, D_{L}9 to D_{NUM}0, D_{L}15 to D_{O}0, D_{L}7 to D_{PL}0, D_{L}11 to D_{RL}0, D_{L}2 to D_{Spare}1, D_{L}3 to D_{S}0, D_{L}4 to D_{S}1, D_{L}5 to D_{TL}0, D_{L}8 to D_{W}0, H1 to H0, K1 to K0, Number_Bar1 to Number_Bar0, Number_Bar2 to Number_Bar1, Number_Bar3 to Number_Bar2, Number_Bar4 to Number_Bar3, Number_Bar5 to Number_Bar4, Number_Bar6 to Number_Bar5, O1 to O0, P_{L}1 to P_{L}0, R_{L}1 to R_{L}0, S1 to S0, S2 to S1, Spare1 to Spare0, Spare2 to Spare1, T_{L}1 to T_{L}0, W1 to W0
Changed lines of the file:
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@@
 		(on_board yes)
 		(dnp no)
-		(property "Reference" "D_{L}8"
+		(property "Reference" "D_{W}0"
 			(at 166.37 95.25 0)
 			(effects
@@
 		(dnp no)
 		(fields_autoplaced yes)
-		(property "Reference" "Number_Bar4"
+		(property "Reference" "Number_Bar3"
 			(at 152.4 50.8 0)
 			(effects
@@
 		(on_board yes)
 		(dnp no)
-		(property "Reference" "D_{L}7"
+		(property "Reference" "D_{PL}0"
 			(at 166.37 73.66 0)
 			(effects
@@
 		(on_board yes)
 		(dnp no)
-		(property "Reference" "Spare1"
+		(property "Reference" "Spare0"
 			(at 30.48 72.39 0)
 			(effects
@@
 		(on_board yes)
 		(dnp no)
-		(property "Reference" "D_{L}10"
+		(property "Reference" "D_{H}0"
 			(at 207.01 73.66 0)
 			(effects
@@
 		(on_board yes)
 		(dnp no)
-		(property "Reference" "P_{L}1"
+		(property "Reference" "P_{L}0"
 			(at 152.4 72.39 0)
 			(effects
@@
 		(on_board yes)
 		(dnp no)
-		(property "Reference" "K1"
+		(property "Reference" "K0"
 			(at 111.76 93.98 0)
 			(effects
@@
 		(on_board yes)
 		(dnp no)
-		(property "Reference" "D_{L}14"
+		(property "Reference" "D_{AS}1"
 			(at 246.38 95.25 0)
 			(effects
@@
 		(dnp no)
 		(fields_autoplaced yes)
-		(property "Reference" "Number_Bar3"
+		(property "Reference" "Number_Bar2"
 			(at 110.49 50.8 0)
 			(effects
@@
 		(on_board yes)
 		(dnp no)
-		(property "Reference" "D_{L}9"
+		(property "Reference" "D_{NUM}0"
 			(at 167.64 41.91 0)
 			(effects
@@
 		(on_board yes)
 		(dnp no)
-		(property "Reference" "Spare2"
+		(property "Reference" "Spare1"
 			(at 30.48 93.98 0)
 			(effects
@@
 		(on_board yes)
 		(dnp no)
-		(property "Reference" "S2"
+		(property "Reference" "S1"
 			(at 71.12 93.98 0)
 			(effects
@@
 		(on_board yes)
 		(dnp no)
-		(property "Reference" "D_{L}3"
+		(property "Reference" "D_{S}0"
 			(at 85.09 73.66 0)
 			(effects
@@
 		(on_board yes)
 		(dnp no)
-		(property "Reference" "A1"
+		(property "Reference" "A0"
 			(at 193.04 115.57 0)
 			(effects
@@
 		(on_board yes)
 		(dnp no)
-		(property "Reference" "D_{L}13"
+		(property "Reference" "D_{As}0"
 			(at 246.38 73.66 0)
 			(effects
@@
 		(on_board yes)
 		(dnp no)
-		(property "Reference" "R_{L}1"
+		(property "Reference" "R_{L}0"
 			(at 193.04 93.98 0)
 			(effects
@@
 		(on_board yes)
 		(dnp no)
-		(property "Reference" "W1"
+		(property "Reference" "W0"
 			(at 152.4 93.98 0)
 			(effects
@@
 		(on_board yes)
 		(dnp no)
-		(property "Reference" "D_{L}6"
+		(property "Reference" "D_{K}0"
 			(at 125.73 95.25 0)
 			(effects
@@
 		(on_board yes)
 		(dnp no)
-		(property "Reference" "Asterisk1"
+		(property "Reference" "Asterisk0"
 			(at 232.41 72.39 0)
 			(effects
@@
 		(on_board yes)
 		(dnp no)
-		(property "Reference" "D_{L}4"
+		(property "Reference" "D_{S}1"
 			(at 85.09 95.25 0)
 			(effects
@@
 		(on_board yes)
 		(dnp no)
-		(property "Reference" "D_{L}5"
+		(property "Reference" "D_{TL}0"
 			(at 125.73 73.66 0)
 			(effects
@@
 		(dnp no)
 		(fields_autoplaced yes)
-		(property "Reference" "Number_Bar2"
+		(property "Reference" "Number_Bar1"
 			(at 72.39 50.8 0)
 			(effects
@@
 		(on_board yes)
 		(dnp no)
-		(property "Reference" "Asterisk2"
+		(property "Reference" "Asterisk1"
 			(at 232.41 93.98 0)
 			(effects
@@
 		(on_board yes)
 		(dnp no)
-		(property "Reference" "T_{L}1"
+		(property "Reference" "T_{L}0"
 			(at 111.76 72.39 0)
 			(effects
@@
 		(on_board yes)
 		(dnp no)
-		(property "Reference" "D_{L}12"
+		(property "Reference" "D_{A}0"
 			(at 207.01 116.84 0)
 			(effects
@@
 		(on_board yes)
 		(dnp no)
-		(property "Reference" "D_{L}15"
+		(property "Reference" "D_{O}0"
 			(at 246.38 116.84 0)
 			(effects
@@
 		(on_board yes)
 		(dnp no)
-		(property "Reference" "D_{L}11"
+		(property "Reference" "D_{RL}0"
 			(at 207.01 95.25 0)
 			(effects
@@
 		(on_board yes)
 		(dnp no)
-		(property "Reference" "S1"
+		(property "Reference" "S0"
 			(at 71.12 72.39 0)
 			(effects
@@
 		(on_board yes)
 		(dnp no)
-		(property "Reference" "H1"
+		(property "Reference" "H0"
 			(at 193.04 72.39 0)
 			(effects
@@
 		(on_board yes)
 		(dnp no)
-		(property "Reference" "O1"
+		(property "Reference" "O0"
 			(at 232.41 115.57 0)
 			(effects
@@
 		(dnp no)
 		(fields_autoplaced yes)
-		(property "Reference" "Number_Bar1"
+		(property "Reference" "Number_Bar0"
 			(at 30.48 50.8 0)
 			(effects
@@
 		(on_board yes)
 		(dnp no)
-		(property "Reference" "D_{L}2"
+		(property "Reference" "D_{Spare}1"
 			(at 44.45 95.25 0)
 			(effects
@@
 		(dnp no)
 		(fields_autoplaced yes)
-		(property "Reference" "Number_Bar6"
+		(property "Reference" "Number_Bar5"
 			(at 232.41 50.8 0)
 			(effects
@@
 		(dnp no)
 		(fields_autoplaced yes)
-		(property "Reference" "Number_Bar5"
+		(property "Reference" "Number_Bar4"
 			(at 191.77 50.8 0)
 			(effects
