File: right_hand_keys.kicad_sch (KiCad schematic)
At the start: 40 parts

Commit message: Label keys
Parts:
- renumbered Key26 to Asterisk2, Key27 to Asterisk3, Key22 to B, Key15 to D, Key28 to E, Key23 to F, Key20 to G, Key19 to L, Number_Bar7 to Number_Bar10, Number_Bar6 to Number_Bar11, Number_Bar11 to Number_Bar6, Number_Bar10 to Number_Bar7, Number_Bar9 to Number_Bar8, Number_Bar8 to Number_Bar9, Key21 to P, Key24 to R, Key18 to S, Key17 to T, Key25 to U, Key16 to Z
Changed lines of the file:
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@@
 		(dnp no)
 		(fields_autoplaced yes)
-		(property "Reference" "Number_Bar9"
+		(property "Reference" "Number_Bar8"
 			(at 140.97 50.8 0)
 			(effects
@@
 			(project "portable_steno"
 				(path "/06a6eca0-edda-4cc0-a23f-017602e67f07/99f3b279-b2b0-4dd5-ab05-9b518546ce95/f651b724-284b-4a82-a638-8f4a85d8d53c"
-					(reference "Number_Bar9")
+					(reference "Number_Bar8")
 					(unit 1)
 				)
@@
 		(on_board yes)
 		(dnp no)
-		(property "Reference" "Key15"
+		(property "Reference" "D"
 			(at 262.89 72.39 0)
 			(effects
@@
 			(project "portable_steno"
 				(path "/06a6eca0-edda-4cc0-a23f-017602e67f07/99f3b279-b2b0-4dd5-ab05-9b518546ce95/f651b724-284b-4a82-a638-8f4a85d8d53c"
-					(reference "Key15")
+					(reference "D")
 					(unit 1)
 				)
@@
 		(on_board yes)
 		(dnp no)
-		(property "Reference" "Key21"
+		(property "Reference" "P"
 			(at 140.97 72.39 0)
 			(effects
@@
 			(project "portable_steno"
 				(path "/06a6eca0-edda-4cc0-a23f-017602e67f07/99f3b279-b2b0-4dd5-ab05-9b518546ce95/f651b724-284b-4a82-a638-8f4a85d8d53c"
-					(reference "Key21")
+					(reference "P")
 					(unit 1)
 				)
@@
 		(on_board yes)
 		(dnp no)
-		(property "Reference" "Key20"
+		(property "Reference" "G"
 			(at 181.61 93.98 0)
 			(effects
@@
 			(project "portable_steno"
 				(path "/06a6eca0-edda-4cc0-a23f-017602e67f07/99f3b279-b2b0-4dd5-ab05-9b518546ce95/f651b724-284b-4a82-a638-8f4a85d8d53c"
-					(reference "Key20")
+					(reference "G")
 					(unit 1)
 				)
@@
 		(dnp no)
 		(fields_autoplaced yes)
-		(property "Reference" "Number_Bar8"
+		(property "Reference" "Number_Bar9"
 			(at 182.88 50.8 0)
 			(effects
@@
 			(project "portable_steno"
 				(path "/06a6eca0-edda-4cc0-a23f-017602e67f07/99f3b279-b2b0-4dd5-ab05-9b518546ce95/f651b724-284b-4a82-a638-8f4a85d8d53c"
-					(reference "Number_Bar8")
+					(reference "Number_Bar9")
 					(unit 1)
 				)
@@
 		(on_board yes)
 		(dnp no)
-		(property "Reference" "Key16"
+		(property "Reference" "Z"
 			(at 262.89 93.98 0)
 			(effects
@@
 			(project "portable_steno"
 				(path "/06a6eca0-edda-4cc0-a23f-017602e67f07/99f3b279-b2b0-4dd5-ab05-9b518546ce95/f651b724-284b-4a82-a638-8f4a85d8d53c"
-					(reference "Key16")
+					(reference "Z")
 					(unit 1)
 				)
@@
 		(on_board yes)
 		(dnp no)
-		(property "Reference" "Key18"
+		(property "Reference" "S"
 			(at 222.25 93.98 0)
 			(effects
@@
 			(project "portable_steno"
 				(path "/06a6eca0-edda-4cc0-a23f-017602e67f07/99f3b279-b2b0-4dd5-ab05-9b518546ce95/f651b724-284b-4a82-a638-8f4a85d8d53c"
-					(reference "Key18")
+					(reference "S")
 					(unit 1)
 				)
@@
 		(on_board yes)
 		(dnp no)
-		(property "Reference" "Key25"
+		(property "Reference" "U"
 			(at 100.33 115.57 0)
 			(effects
@@
 			(project "portable_steno"
 				(path "/06a6eca0-edda-4cc0-a23f-017602e67f07/99f3b279-b2b0-4dd5-ab05-9b518546ce95/f651b724-284b-4a82-a638-8f4a85d8d53c"
-					(reference "Key25")
+					(reference "U")
 					(unit 1)
 				)
@@
 		(on_board yes)
 		(dnp no)
-		(property "Reference" "Key24"
+		(property "Reference" "R"
 			(at 100.33 93.98 0)
 			(effects
@@
 			(project "portable_steno"
 				(path "/06a6eca0-edda-4cc0-a23f-017602e67f07/99f3b279-b2b0-4dd5-ab05-9b518546ce95/f651b724-284b-4a82-a638-8f4a85d8d53c"
-					(reference "Key24")
+					(reference "R")
 					(unit 1)
 				)
@@
 		(on_board yes)
 		(dnp no)
-		(property "Reference" "Key22"
+		(property "Reference" "B"
 			(at 140.97 93.98 0)
 			(effects
@@
 			(project "portable_steno"
 				(path "/06a6eca0-edda-4cc0-a23f-017602e67f07/99f3b279-b2b0-4dd5-ab05-9b518546ce95/f651b724-284b-4a82-a638-8f4a85d8d53c"
-					(reference "Key22")
+					(reference "B")
 					(unit 1)
 				)
@@
 		(on_board yes)
 		(dnp no)
-		(property "Reference" "Key26"
+		(property "Reference" "Asterisk2"
 			(at 60.96 72.39 0)
 			(effects
@@
 			(project "portable_steno"
 				(path "/06a6eca0-edda-4cc0-a23f-017602e67f07/99f3b279-b2b0-4dd5-ab05-9b518546ce95/f651b724-284b-4a82-a638-8f4a85d8d53c"
-					(reference "Key26")
+					(reference "Asterisk2")
 					(unit 1)
 				)
@@
 		(dnp no)
 		(fields_autoplaced yes)
-		(property "Reference" "Number_Bar7"
+		(property "Reference" "Number_Bar10"
 			(at 220.98 50.8 0)
 			(effects
@@
 			(project "portable_steno"
 				(path "/06a6eca0-edda-4cc0-a23f-017602e67f07/99f3b279-b2b0-4dd5-ab05-9b518546ce95/f651b724-284b-4a82-a638-8f4a85d8d53c"
-					(reference "Number_Bar7")
+					(reference "Number_Bar10")
 					(unit 1)
 				)
@@
 		(on_board yes)
 		(dnp no)
-		(property "Reference" "Key27"
+		(property "Reference" "Asterisk3"
 			(at 60.96 93.98 0)
 			(effects
@@
 			(project "portable_steno"
 				(path "/06a6eca0-edda-4cc0-a23f-017602e67f07/99f3b279-b2b0-4dd5-ab05-9b518546ce95/f651b724-284b-4a82-a638-8f4a85d8d53c"
-					(reference "Key27")
+					(reference "Asterisk3")
 					(unit 1)
 				)
@@
 		(on_board yes)
 		(dnp no)
-		(property "Reference" "Key19"
+		(property "Reference" "L"
 			(at 181.61 72.39 0)
 			(effects
@@
 			(project "portable_steno"
 				(path "/06a6eca0-edda-4cc0-a23f-017602e67f07/99f3b279-b2b0-4dd5-ab05-9b518546ce95/f651b724-284b-4a82-a638-8f4a85d8d53c"
-					(reference "Key19")
+					(reference "L")
 					(unit 1)
 				)
@@
 		(on_board yes)
 		(dnp no)
-		(property "Reference" "Key17"
+		(property "Reference" "T"
 			(at 222.25 72.39 0)
 			(effects
@@
 			(project "portable_steno"
 				(path "/06a6eca0-edda-4cc0-a23f-017602e67f07/99f3b279-b2b0-4dd5-ab05-9b518546ce95/f651b724-284b-4a82-a638-8f4a85d8d53c"
-					(reference "Key17")
+					(reference "T")
 					(unit 1)
 				)
@@
 		(on_board yes)
 		(dnp no)
-		(property "Reference" "Key23"
+		(property "Reference" "F"
 			(at 100.33 72.39 0)
 			(effects
@@
 			(project "portable_steno"
 				(path "/06a6eca0-edda-4cc0-a23f-017602e67f07/99f3b279-b2b0-4dd5-ab05-9b518546ce95/f651b724-284b-4a82-a638-8f4a85d8d53c"
-					(reference "Key23")
+					(reference "F")
 					(unit 1)
 				)
@@
 		(on_board yes)
 		(dnp no)
-		(property "Reference" "Key28"
+		(property "Reference" "E"
 			(at 60.96 115.57 0)
 			(effects
@@
 			(project "portable_steno"
 				(path "/06a6eca0-edda-4cc0-a23f-017602e67f07/99f3b279-b2b0-4dd5-ab05-9b518546ce95/f651b724-284b-4a82-a638-8f4a85d8d53c"
-					(reference "Key28")
+					(reference "E")
 					(unit 1)
 				)
@@
 		(dnp no)
 		(fields_autoplaced yes)
-		(property "Reference" "Number_Bar6"
+		(property "Reference" "Number_Bar11"
 			(at 262.89 50.8 0)
 			(effects
@@
 			(project "portable_steno"
 				(path "/06a6eca0-edda-4cc0-a23f-017602e67f07/99f3b279-b2b0-4dd5-ab05-9b518546ce95/f651b724-284b-4a82-a638-8f4a85d8d53c"
-					(reference "Number_Bar6")
+					(reference "Number_Bar11")
 					(unit 1)
 				)
@@
 		(dnp no)
 		(fields_autoplaced yes)
-		(property "Reference" "Number_Bar11"
+		(property "Reference" "Number_Bar6"
 			(at 60.96 50.8 0)
 			(effects
@@
 			(project "portable_steno"
 				(path "/06a6eca0-edda-4cc0-a23f-017602e67f07/99f3b279-b2b0-4dd5-ab05-9b518546ce95/f651b724-284b-4a82-a638-8f4a85d8d53c"
-					(reference "Number_Bar11")
+					(reference "Number_Bar6")
 					(unit 1)
 				)
@@
 		(dnp no)
 		(fields_autoplaced yes)
-		(property "Reference" "Number_Bar10"
+		(property "Reference" "Number_Bar7"
 			(at 101.6 50.8 0)
 			(effects
@@
 			(project "portable_steno"
 				(path "/06a6eca0-edda-4cc0-a23f-017602e67f07/99f3b279-b2b0-4dd5-ab05-9b518546ce95/f651b724-284b-4a82-a638-8f4a85d8d53c"
-					(reference "Number_Bar10")
+					(reference "Number_Bar7")
 					(unit 1)
 				)

Commit message: Design power
Parts:
- D16, D17, D18, D19, D20, D21, D22, D23, D24, D25, D26, D27, D28, D29, D30, D32, D34, D36, D38, D40: footprint Diode_SMD:D_SOD-123 -> Diode_SMD:D_SOD-323
Other:
- title: Port Plover -> Stenoswitch
Changed lines of the file:
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@@
 	(paper "A4")
 	(title_block
-		(title "Port Plover")
-		(date "2025-07-28")
+		(title "Stenoswitch")
 		(rev "0.1")
 		(company "https://github.com/Bennett-Petzold/port_plover")
@@
 			)
 		)
-		(property "Footprint" "Diode_SMD:D_SOD-123"
+		(property "Footprint" "Diode_SMD:D_SOD-323"
 			(at 127 97.155 0)
 			(effects
@@
 			)
 		)
-		(property "Footprint" "Diode_SMD:D_SOD-123"
+		(property "Footprint" "Diode_SMD:D_SOD-323"
 			(at 127 75.565 0)
 			(effects
@@
 			)
 		)
-		(property "Footprint" "Diode_SMD:D_SOD-123"
+		(property "Footprint" "Diode_SMD:D_SOD-323"
 			(at 207.01 53.975 0)
 			(effects
@@
 			)
 		)
-		(property "Footprint" "Diode_SMD:D_SOD-123"
+		(property "Footprint" "Diode_SMD:D_SOD-323"
 			(at 86.36 75.565 0)
 			(effects
@@
 			)
 		)
-		(property "Footprint" "Diode_SMD:D_SOD-123"
+		(property "Footprint" "Diode_SMD:D_SOD-323"
 			(at 46.99 97.155 0)
 			(effects
@@
 			)
 		)
-		(property "Footprint" "Diode_SMD:D_SOD-123"
+		(property "Footprint" "Diode_SMD:D_SOD-323"
 			(at 248.92 75.565 0)
 			(effects
@@
 			)
 		)
-		(property "Footprint" "Diode_SMD:D_SOD-123"
+		(property "Footprint" "Diode_SMD:D_SOD-323"
 			(at 208.28 75.565 0)
 			(effects
@@
 			)
 		)
-		(property "Footprint" "Diode_SMD:D_SOD-123"
+		(property "Footprint" "Diode_SMD:D_SOD-323"
 			(at 127 53.975 0)
 			(effects
@@
 			)
 		)
-		(property "Footprint" "Diode_SMD:D_SOD-123"
+		(property "Footprint" "Diode_SMD:D_SOD-323"
 			(at 46.99 75.565 0)
 			(effects
@@
 			)
 		)
-		(property "Footprint" "Diode_SMD:D_SOD-123"
+		(property "Footprint" "Diode_SMD:D_SOD-323"
 			(at 167.64 97.155 0)
 			(effects
@@
 			)
 		)
-		(property "Footprint" "Diode_SMD:D_SOD-123"
+		(property "Footprint" "Diode_SMD:D_SOD-323"
 			(at 208.28 97.155 0)
 			(effects
@@
 			)
 		)
-		(property "Footprint" "Diode_SMD:D_SOD-123"
+		(property "Footprint" "Diode_SMD:D_SOD-323"
 			(at 167.64 75.565 0)
 			(effects
@@
 			)
 		)
-		(property "Footprint" "Diode_SMD:D_SOD-123"
+		(property "Footprint" "Diode_SMD:D_SOD-323"
 			(at 248.92 53.975 0)
 			(effects
@@
 			)
 		)
-		(property "Footprint" "Diode_SMD:D_SOD-123"
+		(property "Footprint" "Diode_SMD:D_SOD-323"
 			(at 46.99 53.975 0)
 			(effects
@@
 			)
 		)
-		(property "Footprint" "Diode_SMD:D_SOD-123"
+		(property "Footprint" "Diode_SMD:D_SOD-323"
 			(at 86.36 118.745 0)
 			(effects
@@
 			)
 		)
-		(property "Footprint" "Diode_SMD:D_SOD-123"
+		(property "Footprint" "Diode_SMD:D_SOD-323"
 			(at 168.91 53.975 0)
 			(effects
@@
 			)
 		)
-		(property "Footprint" "Diode_SMD:D_SOD-123"
+		(property "Footprint" "Diode_SMD:D_SOD-323"
 			(at 46.99 118.745 0)
 			(effects
@@
 			)
 		)
-		(property "Footprint" "Diode_SMD:D_SOD-123"
+		(property "Footprint" "Diode_SMD:D_SOD-323"
 			(at 86.36 97.155 0)
 			(effects
@@
 			)
 		)
-		(property "Footprint" "Diode_SMD:D_SOD-123"
+		(property "Footprint" "Diode_SMD:D_SOD-323"
 			(at 248.92 97.155 0)
 			(effects
@@
 			)
 		)
-		(property "Footprint" "Diode_SMD:D_SOD-123"
+		(property "Footprint" "Diode_SMD:D_SOD-323"
 			(at 87.63 53.975 0)
 			(effects

Commit message: Remove unnecessary diodes
Parts:
- removed B, D, E, F, G, L, P, R, S, T, U, Z: SW_Push, PCM_Switch_Keyboard_Cherry_MX:SW_Cherry_MX_PCB, symbol Switch:SW_Push
- removed D16, D17, D18, D19, D20, D21, D22, D23, D24, D25, D26, D27, D28, D29, D30, D32, D34, D36, D38, D40: 1N4148WX-TP, Diode_SMD:D_SOD-323, symbol Diode:1N4148W
- added B0, D0, E0, F0, G0, L0, P_{R}0, R_{R}0, S2, T_{R}0, U0, Z0: SW_Push, PCM_Switch_Keyboard_Cherry_MX:SW_Cherry_MX_PCB, symbol Switch:SW_Push
- added D_{R}0, D_{R}1, D_{R}10, D_{R}11, D_{R}12, D_{R}13, D_{R}14, D_{R}2, D_{R}3, D_{R}4, D_{R}5, D_{R}6, D_{R}7, D_{R}8, D_{R}9: 1N4148WX-TP, Diode_SMD:D_SOD-323, symbol Diode:1N4148W
Connections:
- net Columns0: now also D_{R}11.1 (K), D_{R}12.1 (K), D_{R}14.1 (K)
- net Columns1: now also D_{R}10.1 (K), D_{R}13.1 (K), D_{R}9.1 (K)
- net Columns2: now also D_{R}6.1 (K), D_{R}7.1 (K), D_{R}8.1 (K)
- net Columns3: now also D_{R}3.1 (K), D_{R}4.1 (K), D_{R}5.1 (K)
- net Columns4: now also D_{R}0.1 (K), D_{R}1.1 (K), D_{R}2.1 (K)
- net Rows0: now also F0.1, L0.1, P_{R}0.1, T_{R}0.1
- net Rows1: now also B0.1, G0.1, R_{R}0.1, S2.1
- net Rows2: now also D0.1, E0.1, U0.1, Z0.1
- net at Number_Bar8.2: now also Number_Bar10.2, Number_Bar11.2, Number_Bar6.2, Number_Bar7.2, Number_Bar9.2, D_{R}6.2 (A)
- net at Asterisk3.2: now also D_{R}1.2 (A)
- net at Asterisk2.2: now also D_{R}0.2 (A)
- new net: D_{R}9.2 (A), L0.2
- new net: D_{R}10.2 (A), G0.2
- new net: B0.2, D_{R}8.2 (A)
- new net: D_{R}5.2 (A), U0.2
- new net: D_{R}14.2 (A), Z0.2
- new net: D0.2, D_{R}13.2 (A)
- new net: D_{R}2.2 (A), E0.2
- new net: D_{R}11.2 (A), T_{R}0.2
- new net: D_{R}12.2 (A), S2.2
- new net: D_{R}7.2 (A), P_{R}0.2
- new net: D_{R}3.2 (A), F0.2
- new net: D_{R}4.2 (A), R_{R}0.2

Commit message: Init right and left PCBs
Parts:
- renumbered Asterisk2 to Asterisk1, Asterisk3 to Asterisk2, B0 to B1, D0 to D1, D_{R}0 to D_{R}1, D_{R}9 to D_{R}10, D_{R}10 to D_{R}11, D_{R}11 to D_{R}12, D_{R}12 to D_{R}13, D_{R}13 to D_{R}14, D_{R}14 to D_{R}15, D_{R}1 to D_{R}2, D_{R}2 to D_{R}3, D_{R}3 to D_{R}4, D_{R}4 to D_{R}5, D_{R}5 to D_{R}6, D_{R}6 to D_{R}7, D_{R}7 to D_{R}8, D_{R}8 to D_{R}9, E0 to E1, F0 to F1, G0 to G1, L0 to L1, Number_Bar6 to Number_Bar1, Number_Bar7 to Number_Bar2, Number_Bar8 to Number_Bar3, Number_Bar9 to Number_Bar4, Number_Bar10 to Number_Bar5, Number_Bar11 to Number_Bar6, P_{R}0 to P_{R}1, R_{R}0 to R_{R}1, S2 to S1, T_{R}0 to T_{R}1, U0 to U1, Z0 to Z1

Commit message: Rename keyswitch diodes
Parts:
- renumbered Asterisk1 to Asterisk2, Asterisk2 to Asterisk3, B1 to B0, D1 to D0, D_{R}1 to D_{AS}2, D_{R}2 to D_{AS}3, D_{R}9 to D_{B}0, D_{R}14 to D_{D}0, D_{R}3 to D_{E}0, D_{R}4 to D_{F}0, D_{R}11 to D_{G}0, D_{R}10 to D_{L}0, D_{R}7 to D_{NUM}1, D_{R}8 to D_{PR}0, D_{R}5 to D_{RR}0, D_{R}13 to D_{S}2, D_{R}12 to D_{TR}0, D_{R}6 to D_{U}0, D_{R}15 to D_{Z}0, E1 to E0, F1 to F0, G1 to G0, L1 to L0, Number_Bar5 to Number_Bar10, Number_Bar6 to Number_Bar11, Number_Bar1 to Number_Bar6, Number_Bar2 to Number_Bar7, Number_Bar3 to Number_Bar8, Number_Bar4 to Number_Bar9, P_{R}1 to P_{R}0, R_{R}1 to R_{R}0, S1 to S2, T_{R}1 to T_{R}0, U1 to U0, Z1 to Z0
