File: left_hand/left_hand.kicad_pcb (KiCad board)
At the start: 2 copper layers, 36 parts, among them K1 SW_Push

Commit message: Layout left hand side
Parts:
- D_{AS}1: renamed from D_{L}14; moved to B.Cu
- D_{As}0: renamed from D_{L}13; moved to B.Cu
- D_{A}0: renamed from D_{L}12; moved to B.Cu
- D_{H}0: renamed from D_{L}10; moved to B.Cu
- D_{K}0: renamed from D_{L}6; moved to B.Cu
- D_{NUM}0: renamed from D_{L}9; moved to B.Cu
- D_{O}0: renamed from D_{L}15; moved to B.Cu
- D_{PL}0: renamed from D_{L}7; moved to B.Cu
- D_{RL}0: renamed from D_{L}11; moved to B.Cu
- D_{Spare}0: renamed from D_{L}1; moved to B.Cu
- D_{Spare}1: renamed from D_{L}2; moved to B.Cu
- D_{S}0: renamed from D_{L}3; moved to B.Cu
- D_{S}1: renamed from D_{L}4; moved to B.Cu
- D_{TL}0: renamed from D_{L}5; moved to B.Cu
- D_{W}0: renamed from D_{L}8; moved to B.Cu
- moved A0 136.2 mm to (188.6, 143.3)
- moved D_{NUM}0 120.9 mm to (196.6, 71.0), turned to -90 degrees
- moved D_{O}0 112.6 mm to (199.0, 138.0), turned to -90 degrees
- moved D_{As}0 109.9 mm to (196.7, 90.2), turned to -90 degrees
- moved D_{AS}1 108.3 mm to (196.8, 109.1), turned to -90 degrees
- moved Asterisk1 107.1 mm to (188.6, 114.7)
- moved Asterisk0 106.2 mm to (188.6, 95.7)
- moved O0 100.4 mm to (207.6, 143.3)
- moved D_{H}0 97.8 mm to (177.8, 90.1), turned to -90 degrees
- moved D_{A}0 96.6 mm to (180.0, 137.7), turned to -90 degrees
- moved D_{RL}0 94.4 mm to (177.8, 109.1), turned to -90 degrees
- moved Spare1 93.5 mm to (74.2, 127.4)
- moved Spare0 91.4 mm to (74.2, 108.4)
- moved H0 84.1 mm to (169.5, 95.7)
- moved D_{PL}0 75.5 mm to (152.4, 77.4), turned to -90 degrees
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- renumbered A1 to A0, Asterisk1 to Asterisk0, Asterisk2 to Asterisk1, H1 to H0, K1 to K0, Number_Bar1 to Number_Bar0, Number_Bar2 to Number_Bar1, Number_Bar3 to Number_Bar2, Number_Bar4 to Number_Bar3, Number_Bar5 to Number_Bar4, Number_Bar6 to Number_Bar5, O1 to O0, P_{L}1 to P_{L}0, R_{L}1 to R_{L}0, S1 to S0, S2 to S1, Spare1 to Spare0, Spare2 to Spare1, T_{L}1 to T_{L}0, W1 to W0
Connections:
- Left_Plug1 pad 1: /Columns0 -> /Columns3
- Left_Plug1 pad 2: /Columns1 -> /Columns0
- Left_Plug1 pad 3: /Columns2 -> /Columns1
- Left_Plug1 pad 4: /Columns3 -> /Columns2
- Left_Plug1 pad 6: /Rows0 -> /Rows1
- Left_Plug1 pad 7: /Rows1 -> /Rows0
Routing:
- net /Rows2: track 0.00 -> 331.6 mm
- net Net-(D_{NUM}0-A): track 0.00 -> 286.3 mm
- net /Columns0: track 0.00 -> 183.2 mm
- net /Columns1: track 0.00 -> 174.5 mm
- net /Rows1: track 0.00 -> 152.3 mm
- net /Rows0: track 0.00 -> 138.7 mm
- net /Columns3: track 0.00 -> 95.9 mm
- net /Columns2: track 0.00 -> 90.3 mm
- net /Columns4: track 0.00 -> 63.1 mm
- net Net-(D_{O}0-A): track 0.00 -> 11.5 mm
- net Net-(D_{A}0-A): track 0.00 -> 11.3 mm
- net Net-(D_{W}0-A): track 0.00 -> 6.01 mm
- net Net-(D_{TL}0-A): track 0.00 -> 5.97 mm
- net Net-(D_{PL}0-A): track 0.00 -> 5.97 mm
- net Net-(D_{K}0-A): track 0.00 -> 5.97 mm
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Other:
- board outline added: 160 x 110 mm
- board text added: "Stenoswitch Left Hand v0.1"
