File: right_hand/battery.kicad_sch (KiCad schematic)
At the start: 43 parts

Commit message: Rework right hand
Connections:
- net at BAT_MIN0.2, R_{Pullup}0.1, STORE_EN0.2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: now also BAT_EN0.1; no longer BAT_EN0.2
- net at Battery_Charger0.5 (BATT), Battery_Monitor0.C2 (SRX), CHRG_Shunt0.1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: now also BAT_EN0.2; no longer BAT_EN0.1
