File: pcb/left_hand/left_hand.kicad_pcb (KiCad board)
At the start: 2 copper layers, 150 x 105 mm, 43 parts, among them K0 SW_Push

Commit message: Make left hand pads larger
Parts:
- D_{AS}1, D_{As}0, D_{A}0, D_{H}0, D_{K}0, D_{NUM}0, D_{O}0, D_{PL}0, D_{RL}0, D_{Spare}0, D_{Spare}1, D_{S}0, D_{S}1, D_{TL}0, D_{W}0: footprint Diode_SMD:D_SOD-323 -> Diode_SMD:D_SOD-323_HandSoldering
Other:
- board text added: "Stenoswitch Left Hand v0.3"
- board text removed: "Stenoswitch Left Hand v0.2"
