File: pcb/right_hand.kicad_sch (KiCad schematic)
At the start: 1 part

Commit message: Add DNP for right hand
Parts:
- Right_Plug0: now not fitted
Changed lines of the file:
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@@
 		(in_bom yes)
 		(on_board yes)
-		(dnp no)
+		(dnp yes)
 		(fields_autoplaced yes)
 		(property "Reference" "Right_Plug0"
